File: hardware/dekatron/power.kicad_sch (KiCad schematic)
At the start: 95 parts, among them J101 PWR_IN, J102 NIX_12V, Q101 AOD4185, Q102 AOD5N40, U101 TPS54202, U102 LM66100, U103 LM66100, U104 LM66100, U105 LP2951 (adj. 10 V), U106 LM5156H, U107 TLV3011, U108 TLV3011

Commit message: Phase 1C: place and route the dekatron board (100 x 85 mm, DRC clean)
Placement (tools/gen_pcb.py): new 100 x 85 mm outline (was 120 x 100),
hand anchors for the tripler ladder, HV dividers, anode resistors, LM5156
neighbourhood (rotated 90, fan-out keep-outs), RP2040-Zero power parts and
harness landings; multi-rectangle regions; netlist fields copied onto the
footprints; LM5156 thermal vias at 0.3 mm (OSH Park minimum drill).
Schematic: LM5156 footprint without the 0.2 mm library vias; the HV dummy
load is now off-board (bring-up only).

Routing (tools/route_pcb.py, route_loop.sh): fine-pitch nets first with
reserved escape stubs, raster margins from DRC findings, promote-and-retry
passes, GND pour credited on the bottom layer only, GND repair against the
real fill; pcb_io.py adds GND stitching vias. OSH Park DRU values.

DRC: 0 unconnected, 0 clearance, 0 schematic parity; silkscreen warnings
and the expected U106 library mismatch remain. Fab outputs not generated
yet (silkscreen tidy and review first).

Co-Authored-By: Claude Opus 5.5 <noreply@anthropic.com>
Parts:
- removed R145: 910k, Resistor_THT:R_Axial_DIN0411_L9.9mm_D3.6mm_P15.24mm_Horizontal, symbol Device:R
- U106: footprint Package_SO:Texas_HTSSOP-14-1EP_4.4x5mm_P0.65mm_EP3.4x5mm_Mask3.155x3.255mm_ThermalVias -> Package_SO:Texas_HTSSOP-14-1EP_4.4x5mm_P0.65mm_EP3.4x5mm_Mask3.155x3.255mm
Changed lines of the file:
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@@
 	  (property "Reference" "U106" (at 152.4 183.66 0) (show_name no) (do_not_autoplace no) (effects (font (size 1.27 1.27)) (justify left)))
 	  (property "Value" "LM5156H" (at 152.4 185.26 0) (show_name no) (do_not_autoplace no) (effects (font (size 1.27 1.27)) (justify left)))
-	  (property "Footprint" "Package_SO:Texas_HTSSOP-14-1EP_4.4x5mm_P0.65mm_EP3.4x5mm_Mask3.155x3.255mm_ThermalVias" (at 165.1 200.66 0) (hide yes) (show_name no) (do_not_autoplace no) (effects (font (size 1.27 1.27)) (justify left)))
+	  (property "Footprint" "Package_SO:Texas_HTSSOP-14-1EP_4.4x5mm_P0.65mm_EP3.4x5mm_Mask3.155x3.255mm" (at 165.1 200.66 0) (hide yes) (show_name no) (do_not_autoplace no) (effects (font (size 1.27 1.27)) (justify left)))
 	  (property "Datasheet" "https://www.ti.com/lit/ds/symlink/lm5156h.pdf" (at 165.1 200.66 0) (hide yes) (show_name no) (do_not_autoplace no) (effects (font (size 1.27 1.27)) (justify left)))
 	  (property "Description" "65V Wide Vin non-synchronous Boost/SEPIC/Flyback controller, HTSSOP-14" (at 165.1 200.66 0) (hide yes) (show_name no) (do_not_autoplace no) (effects (font (size 1.27 1.27)) (justify left)))
@@
 	(wire (pts (xy 127 251.46) (xy 152.4 251.46)) (stroke (width 0) (type default)))
 	(wire (pts (xy 152.4 251.46) (xy 177.8 251.46)) (stroke (width 0) (type default)))
-	(wire (pts (xy 177.8 251.46) (xy 205.74 251.46)) (stroke (width 0) (type default)))
-	(wire (pts (xy 205.74 251.46) (xy 256.54 251.46)) (stroke (width 0) (type default)))
+	(wire (pts (xy 177.8 251.46) (xy 256.54 251.46)) (stroke (width 0) (type default)))
 	(wire (pts (xy 256.54 251.46) (xy 266.7 251.46)) (stroke (width 0) (type default)))
 	(label "HV_STACK" (at 127 251.46 0) (effects (font (size 1.27 1.27)) (justify left bottom)))
@@
 	  (pin "1")
 	  (instances (project "dekatron" (path "/b14ce2c4-03a1-5284-8a98-bc460407f799/ffb9d6a6-7c3b-5075-b238-678084eb444d" (reference "#PWRPOWER067") (unit 1))))
-	)
-	(wire (pts (xy 205.74 251.46) (xy 205.74 256.54)) (stroke (width 0) (type default)))
-	(symbol (lib_id "Device:R") (at 205.74 260.35 0) (unit 1) (body_style 1) (exclude_from_sim no) (in_bom yes) (on_board yes) (in_pos_files yes) (dnp yes)
-	  (property "Reference" "R145" (at 208.94 259.35 0) (show_name no) (do_not_autoplace no) (effects (font (size 1.27 1.27)) (justify left)))
-	  (property "Value" "910k" (at 208.94 261.95 0) (show_name no) (do_not_autoplace no) (effects (font (size 1.27 1.27)) (justify left)))
-	  (property "Footprint" "Resistor_THT:R_Axial_DIN0411_L9.9mm_D3.6mm_P15.24mm_Horizontal" (at 205.74 260.35 0) (hide yes) (show_name no) (do_not_autoplace no) (effects (font (size 1.27 1.27)) (justify left)))
-	  (property "Datasheet" "" (at 205.74 260.35 0) (hide yes) (show_name no) (do_not_autoplace no) (effects (font (size 1.27 1.27)) (justify left)))
-	  (property "Description" "Resistor" (at 205.74 260.35 0) (hide yes) (show_name no) (do_not_autoplace no) (effects (font (size 1.27 1.27)) (justify left)))
-	  (property "Function" "HV dummy load (bring-up only, LK4 open)" (at 205.74 260.35 0) (hide yes) (show_name no) (do_not_autoplace no) (effects (font (size 1.27 1.27)) (justify left)))
-	  (property "MPN" "HVR3700009103FR500" (at 205.74 260.35 0) (hide yes) (show_name no) (do_not_autoplace no) (effects (font (size 1.27 1.27)) (justify left)))
-	  (property "Manufacturer" "Vishay" (at 205.74 260.35 0) (hide yes) (show_name no) (do_not_autoplace no) (effects (font (size 1.27 1.27)) (justify left)))
-	  (property "Rating" "HVR37: 0.5 W, 3500 V DC, 1 %, 200 ppm/K" (at 205.74 260.35 0) (hide yes) (show_name no) (do_not_autoplace no) (effects (font (size 1.27 1.27)) (justify left)))
-	  (pin "1")
-	  (pin "2")
-	  (instances (project "dekatron" (path "/b14ce2c4-03a1-5284-8a98-bc460407f799/ffb9d6a6-7c3b-5075-b238-678084eb444d" (reference "R145") (unit 1))))
-	)
-	(wire (pts (xy 205.74 264.16) (xy 205.74 266.7)) (stroke (width 0) (type default)))
-	(symbol (lib_id "power:GND") (at 205.74 266.7 0) (unit 1) (body_style 1) (exclude_from_sim no) (in_bom yes) (on_board yes) (in_pos_files yes) (dnp no)
-	  (property "Reference" "#PWRPOWER068" (at 208.94 265.7 0) (hide yes) (show_name no) (do_not_autoplace no) (effects (font (size 1.27 1.27)) (justify left)))
-	  (property "Value" "GND" (at 208.94 268.3 0) (hide yes) (show_name no) (do_not_autoplace no) (effects (font (size 1.27 1.27)) (justify left)))
-	  (property "Footprint" "" (at 205.74 266.7 0) (hide yes) (show_name no) (do_not_autoplace no) (effects (font (size 1.27 1.27)) (justify left)))
-	  (property "Datasheet" "" (at 205.74 266.7 0) (hide yes) (show_name no) (do_not_autoplace no) (effects (font (size 1.27 1.27)) (justify left)))
-	  (property "Description" "Power symbol creates a global label with name \\\"GND\\\" , ground" (at 205.74 266.7 0) (hide yes) (show_name no) (do_not_autoplace no) (effects (font (size 1.27 1.27)) (justify left)))
-	  (pin "1")
-	  (instances (project "dekatron" (path "/b14ce2c4-03a1-5284-8a98-bc460407f799/ffb9d6a6-7c3b-5075-b238-678084eb444d" (reference "#PWRPOWER068") (unit 1))))
 	)
 	(symbol (lib_id "Connector:TestPoint") (at 256.54 251.46 0) (unit 1) (body_style 1) (exclude_from_sim no) (in_bom yes) (on_board yes) (in_pos_files yes) (dnp no)
@@
 	(junction (at 198.12 50.8) (diameter 0) (color 0 0 0 0))
 	(junction (at 200.66 205.74) (diameter 0) (color 0 0 0 0))
-	(junction (at 205.74 251.46) (diameter 0) (color 0 0 0 0))
 	(junction (at 208.28 167.64) (diameter 0) (color 0 0 0 0))
 	(junction (at 213.36 50.8) (diameter 0) (color 0 0 0 0))

Commit message: Swap AOS MOSFETs for Mouser-stocked Infineon parts
Q101 AOD4185 -> IPD50P04P4L-11 (-40 V, 10.6 mohm, 200 A pulsed, VGS +5/-16 V);
input_protect re-run with its resistance: inrush 52.5 A, rail 12.6 V, fuse
I2t 0.089 A2s, VGS -9.97..+0.14 V, reversal blocked.
Q102 AOD5N40 -> IPD50R1K4CE (500 V CoolMOS CE, 1.4 ohm, Vth 2.5-3.5 V): margin
2.56x on the 195 V worst case; figures from distributor listings, flagged to
confirm against Infineon's datasheet.
Same DPAK footprint and pinout; PCB fields updated in place, DRC parity clean.
Fab outputs unchanged (no part values in them).

Co-Authored-By: Claude Opus 5.5 <noreply@anthropic.com>
Parts:
- Q101: value AOD4185 -> IPD50P04P4L-11; MPN AOD4185 -> IPD50P04P4L-11; Manufacturer Alpha & Omega -> Infineon; Rating -40 V, 115 A pulsed -> -40 V, 10.6 mohm, 200 A pulsed, VGS +5/-16 V
- Q102: value AOD5N40 -> IPD50R1K4CE; MPN AOD5N40 -> IPD50R1K4CE; Manufacturer Alpha & Omega -> Infineon; Rating 400 V, 1.6 ohm at 10 V -> 500 V, 1.4 ohm at 10 V
Changed lines of the file:
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@@
 	(symbol (lib_id "Transistor_FET:Q_PMOS_GDS") (at 73.66 53.34 90) (unit 1) (body_style 1) (exclude_from_sim no) (in_bom yes) (on_board yes) (in_pos_files yes) (dnp no)
 	  (property "Reference" "Q101" (at 73.66 46.34 90) (show_name no) (do_not_autoplace no) (effects (font (size 1.27 1.27))))
-	  (property "Value" "AOD4185" (at 73.66 47.94 90) (show_name no) (do_not_autoplace no) (effects (font (size 1.27 1.27))))
+	  (property "Value" "IPD50P04P4L-11" (at 73.66 47.94 90) (show_name no) (do_not_autoplace no) (effects (font (size 1.27 1.27))))
 	  (property "Footprint" "Package_TO_SOT_SMD:TO-252-2" (at 73.66 53.34 90) (hide yes) (show_name no) (do_not_autoplace no) (effects (font (size 1.27 1.27)) (justify left)))
 	  (property "Datasheet" "" (at 73.66 53.34 90) (hide yes) (show_name no) (do_not_autoplace no) (effects (font (size 1.27 1.27)) (justify left)))
 	  (property "Description" "P-MOSFET transistor, gate/drain/source" (at 73.66 53.34 90) (hide yes) (show_name no) (do_not_autoplace no) (effects (font (size 1.27 1.27)) (justify left)))
 	  (property "Function" "Reverse-polarity protection" (at 73.66 53.34 90) (hide yes) (show_name no) (do_not_autoplace no) (effects (font (size 1.27 1.27)) (justify left)))
-	  (property "MPN" "AOD4185" (at 73.66 53.34 90) (hide yes) (show_name no) (do_not_autoplace no) (effects (font (size 1.27 1.27)) (justify left)))
-	  (property "Manufacturer" "Alpha & Omega" (at 73.66 53.34 90) (hide yes) (show_name no) (do_not_autoplace no) (effects (font (size 1.27 1.27)) (justify left)))
-	  (property "Rating" "-40 V, 115 A pulsed" (at 73.66 53.34 90) (hide yes) (show_name no) (do_not_autoplace no) (effects (font (size 1.27 1.27)) (justify left)))
+	  (property "MPN" "IPD50P04P4L-11" (at 73.66 53.34 90) (hide yes) (show_name no) (do_not_autoplace no) (effects (font (size 1.27 1.27)) (justify left)))
+	  (property "Manufacturer" "Infineon" (at 73.66 53.34 90) (hide yes) (show_name no) (do_not_autoplace no) (effects (font (size 1.27 1.27)) (justify left)))
+	  (property "Rating" "-40 V, 10.6 mohm, 200 A pulsed, VGS +5/-16 V" (at 73.66 53.34 90) (hide yes) (show_name no) (do_not_autoplace no) (effects (font (size 1.27 1.27)) (justify left)))
 	  (pin "1")
 	  (pin "2")
@@
 	(symbol (lib_id "Transistor_FET:Q_NMOS_GDS") (at 231.14 193.04 0) (unit 1) (body_style 1) (exclude_from_sim no) (in_bom yes) (on_board yes) (in_pos_files yes) (dnp no)
 	  (property "Reference" "Q102" (at 234.34 192.04 0) (show_name no) (do_not_autoplace no) (effects (font (size 1.27 1.27)) (justify left)))
-	  (property "Value" "AOD5N40" (at 234.34 194.64 0) (show_name no) (do_not_autoplace no) (effects (font (size 1.27 1.27)) (justify left)))
+	  (property "Value" "IPD50R1K4CE" (at 234.34 194.64 0) (show_name no) (do_not_autoplace no) (effects (font (size 1.27 1.27)) (justify left)))
 	  (property "Footprint" "Package_TO_SOT_SMD:TO-252-2" (at 231.14 193.04 0) (hide yes) (show_name no) (do_not_autoplace no) (effects (font (size 1.27 1.27)) (justify left)))
 	  (property "Datasheet" "" (at 231.14 193.04 0) (hide yes) (show_name no) (do_not_autoplace no) (effects (font (size 1.27 1.27)) (justify left)))
 	  (property "Description" "N-MOSFET transistor, gate/drain/source" (at 231.14 193.04 0) (hide yes) (show_name no) (do_not_autoplace no) (effects (font (size 1.27 1.27)) (justify left)))
 	  (property "Function" "HV boost switch" (at 231.14 193.04 0) (hide yes) (show_name no) (do_not_autoplace no) (effects (font (size 1.27 1.27)) (justify left)))
-	  (property "MPN" "AOD5N40" (at 231.14 193.04 0) (hide yes) (show_name no) (do_not_autoplace no) (effects (font (size 1.27 1.27)) (justify left)))
-	  (property "Manufacturer" "Alpha & Omega" (at 231.14 193.04 0) (hide yes) (show_name no) (do_not_autoplace no) (effects (font (size 1.27 1.27)) (justify left)))
-	  (property "Rating" "400 V, 1.6 ohm at 10 V" (at 231.14 193.04 0) (hide yes) (show_name no) (do_not_autoplace no) (effects (font (size 1.27 1.27)) (justify left)))
-	  (pin "1")
-	  (pin "2")
+	  (property "MPN" "IPD50R1K4CE" (at 231.14 193.04 0) (hide yes) (show_name no) (do_not_autoplace no) (effects (font (size 1.27 1.27)) (justify left)))
+	  (property "Manufacturer" "Infineon" (at 231.14 193.04 0) (hide yes) (show_name no) (do_not_autoplace no) (effects (font (size 1.27 1.27)) (justify left)))
+	  (property "Rating" "500 V, 1.4 ohm at 10 V" (at 231.14 193.04 0) (hide yes) (show_name no) (do_not_autoplace no) (effects (font (size 1.27 1.27)) (justify left)))
+	  (pin "1")
+	  (pin "2")
