File: hardware/dekatron/power.kicad_sch (KiCad schematic)
At the start: 94 parts, among them J101 PWR_IN, J102 NIX_12V, Q101 IPD50P04P4L-11, Q102 IPD50R1K4CE, U101 TPS54202, U102 LM66100, U103 LM66100, U104 LM66100, U105 LP2951 (adj. 10 V), U106 LM5156H, U107 TLV3011, U108 TLV3011

Commit message: Use E12 values for the Yageo HHV high-voltage resistors
HHV stock at Mouser follows E12 (2.2M/2.7M stocked, 2.0M/2.4M/332k not).
HHV parts now: 4.7M x2 (feedback, monitor/OVP tops), 2.2M x2 (V_b bleeder,
V_b OVP top), 220k (index), 330k x2 (anode, = D1's 660k design value);
R202 stays 200k (stocked, already ordered). Trims moved to 1206 bottoms:
feedback 10.4k -> 452.9 V (9.53k: 494.2 V); OVP 10.7k -> 548.4 V trip,
HV_SENSE = HV/191.3; V_b OVP 13.7k -> 200.7 V. 500 V anode option 330k +
470k = 800k; off-board dummy load 1M.

Re-simulated: 500 V setting regulates at 494.1 V out of current limit
(tube 368 uA, peaks HV 498 V, V_b 170 V); dark-tube feedback-open fault trips
at 550.3 V, bursts 547.1-549.7 V; open tripler diode holds V_b <= 198.4 V;
discharge < 50 V in 1.94 / 3.93 / 3.47 s. PCB fields synced, ERC/DRC
parity unchanged; footprints and fab files unchanged.

Co-Authored-By: Claude Opus 5.5 <noreply@anthropic.com>
Parts:
- R119: value 2.4M -> 2.2M; MPN HHV-25FT-52-2M4 -> HHV-25FT-52-2M2
- R126: value 4.75M -> 4.7M; MPN HHV-25FT-52-4M75 -> HHV-25FT-52-4M7
- R130: value 10.5k -> 10.4k; Function HV feedback, lower (453.4 V; 9.53k for 500 V) -> HV feedback, lower (452.9 V; 9.53k for 500 V: 494.2 V)
- R131: value 4.64M -> 4.7M; MPN HHV-25FT-52-4M64 -> HHV-25FT-52-4M7
- R135: Function HV monitor / OVP divider, middle (HV_SENSE 2.36 V at 450 V) -> HV monitor / OVP divider, middle (HV_SENSE 2.37 V at 452.9 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
- R140: value 10.5k -> 10.7k; Function HV monitor / OVP divider, lower (OVP trip 551.8 V) -> HV monitor / OVP divider, lower (OVP trip 548.4 V)
- R141: value 2.0M -> 2.2M; MPN HHV-25FT-52-2M -> HHV-25FT-52-2M2
- R143: value 12.4k -> 13.7k; Function V_b OVP divider, lower (trip ~202 V) -> V_b OVP divider, lower (trip 200.7 V)

Commit message: Fix LM66100 reverse blocking (CE to VOUT); 2.7M HV divider tops; re-route
LM66100 (U102-U104): CE was grounded, the datasheet's always-on mode without
reverse-current blocking (SLVSEZ8A 8.3.1). CE now ties to VOUT (8.3.2, always-on
reverse current blocking); unused ST goes to GND as the pin table asks (three
expected ERC open-collector entries).

HV divider tops: HHV-25 4.7M had a 10-week lead time; one stocked 2.7M each
(0.11 W at 550 V). Feedback 2.7M / 5.97k -> 453.3 V (5.49k: 492.8 V); OVP
2.7M / 7.87k / 6.19k -> 544.6 V trip, HV_SENSE = HV/193.0. Re-simulated: 500 V
setting 492.7 V out of current limit (0.34 A of 0.43 A); dark-tube feedback-
open fault trips at 545.8 V; discharge < 50 V in 1.10 / 2.03 / 2.03 s.

Router: LM66100 CE-VOUT laid under the package body before routing, and fixed
GND escape vias for pins 2 and 5 (R301, C108 anchored 0.6 mm clear); 0.03 mm
extra margin against other nets' pads; vias keep 0.25 mm hole-to-hole from
plated holes. Converged on pass 5. DRC: 0 unconnected, 0 clearance, 0 parity;
expected U106 library mismatch and one U107 starved thermal. Fab outputs
regenerated (the previous set was not ordered).

Co-Authored-By: Claude Opus 5.5 <noreply@anthropic.com>
Parts:
- R126, R131: value 4.7M -> 2.7M; MPN HHV-25FT-52-4M7 -> HHV-25FT-52-2M7
- R130: value 10.4k -> 5.97k; Function HV feedback, lower (452.9 V; 9.53k for 500 V: 494.2 V) -> HV feedback, lower (453.3 V; 5.49k for 500 V: 492.8 V)
- R135: value 14.0k -> 7.87k; Function HV monitor / OVP divider, middle (HV_SENSE 2.37 V at 452.9 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 -> HV monitor / OVP divider, middle (HV_SENSE 2.35 V at 453.3 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
- R140: value 10.7k -> 6.19k; Function HV monitor / OVP divider, lower (OVP trip 548.4 V) -> HV monitor / OVP divider, lower (OVP trip 544.6 V)
Connections:
- net 5V_DISP: now also U102.3 (~{CE})
- net 5V_MCU: now also U103.3 (~{CE})
- net 5V_NIX: now also U104.3 (~{CE})
- net GND: now also U102.5 (ST), U103.5 (ST), U104.5 (ST); no longer U102.3 (~{CE}), U103.3 (~{CE}), U104.3 (~{CE})
- no-connect marks 6 -> 3
Other:
- note added: "One LM66100 per external 5 V feed; CE tied to VOUT = always-on reverse-current blocking (datasheet SLVSEZ8A 8.3.2; CE to GND would not block); ST unused, to GND"
- note removed: "One LM66100 per external 5 V feed; CE grounded = always on"

Commit message: WIMA MKS4 film caps (18 x 8 mm) and EEE-FK1V101XP bulk cap; re-route
- C122-C126: WIMA MKS4G034704F00MSSD on the C_Rect L18 W8 P15 footprint;
  C126 moves 0.2 mm down to keep its courtyard off R131.
- C101: Panasonic EEE-FK1V101XP (6.3 x 7.7 mm, 340 mohm). input_protect.cir
  re-run: worst lead 12.0 V / 47.9 A / 0.070 A2s (was 12.5 V / 52.5 A / 0.088).
- Router: 0.05 mm extra clearance to other nets' tracks outside the LM5156
  pin group (DRC found a 0.153 mm VIN_PROT/PGOOD gap from raster error).
- DRC: 0 unconnected / 0 clearance / 0 parity; 2 expected findings.
  Fab outputs regenerated.

Co-Authored-By: Claude Opus 5.5 <noreply@anthropic.com>
Parts:
- C101: footprint Capacitor_SMD:CP_Elec_8x10.5 -> Capacitor_SMD:CP_Elec_6.3x7.7; MPN EEE-FK1V101P -> EEE-FK1V101XP; Rating 35 V, 160 mohm ESR -> 35 V, 340 mohm ESR
- C122, C123, C124, C125, C126: footprint Capacitor_THT:C_Rect_L18.0mm_W7.0mm_P15.00mm_FKS3_FKP3 -> Capacitor_THT:C_Rect_L18.0mm_W8.0mm_P15.00mm_FKS3_FKP3; MPN (none) -> MKS4G034704F00MSSD; Manufacturer (none) -> WIMA

Commit message: Freeze the dekatron BOM to the Mouser order; substitutions; re-route
- ORDERED_PARTS in gen_schematics.py: exact manufacturer part numbers from
  Cart_Oct08_0432PM.xls (committed as the record), overriding design-time MPNs
- Backorder substitutions: TPS54302 (pin-compatible 5 V buck), IPD70R1K4P7S
  (700 V CoolMOS P7, replaces the EOL IPD50R1K4CE), MMSZ5262BT1G, BAT54S RFG
- C301 is the user's F91 tantalum: polarised symbol and EIA 3216-18 footprint
- E24 dividers: HV feedback 2 x 3.0k 0805 (451.0 V; 2 x 2.7k for 500 V),
  OVP lower 6.2k (543.7 V); simulations re-run, docs updated
- Router: exact own-pad clearance, D301 GND escape via kept out of the
  RP2040 no-via area (D301 anchored rotated), 0.3 mm GND repair links
- Full re-route, DRC clean (expected U106 mismatch, one starved thermal);
  fab outputs regenerated

Co-Authored-By: Claude Opus 5.5 <noreply@anthropic.com>
Parts:
- added R144: 3.0k, Resistor_SMD:R_0805_2012Metric, symbol Device:R
- C102, C104, C105, C109, C110, C111, C115, C121, C128, C130: MPN (none) -> CC1206JPX7R9BB104; Manufacturer (none) -> Yageo
- C103, C120: MPN (none) -> CC1210KKX7RGBB106; Manufacturer (none) -> Yageo
- C106, C107: MPN (none) -> MBAST32MSB7226KPNA18; Manufacturer (none) -> Taiyo Yuden
- C108: MPN (none) -> 12065A750JAT2A; Manufacturer (none) -> KYOCERA AVX
- C112, C114: MPN (none) -> 1206DC105MAT2A; Manufacturer (none) -> KYOCERA AVX
- C113: MPN (none) -> CS1206KKX7R8BB225; Manufacturer (none) -> Yageo
- C116: MPN (none) -> CC1206KRX7R8BB473; Manufacturer (none) -> Yageo
- C117: MPN (none) -> 12063C103JAT2A; Manufacturer (none) -> KYOCERA AVX
- C118: MPN (none) -> C1206C101K5GAC7210; Manufacturer (none) -> KEMET
- C119: MPN (none) -> 1206B471K500CT; Manufacturer (none) -> Walsin
- C127, C129: MPN (none) -> 1206N102K501CT; Manufacturer (none) -> Walsin
- D101: Manufacturer (none) -> Diotec Semiconductor
- D102: Manufacturer Littelfuse -> Semtech
- D103, D104, D105, D106, D107: Manufacturer onsemi -> Diotec Semiconductor
- Q101: MPN IPD50P04P4L-11 -> IPD50P04P4L11ATMA2
- Q102: value IPD50R1K4CE -> IPD70R1K4P7S; MPN IPD50R1K4CE -> IPD70R1K4P7SAUMA1; Rating 500 V, 1.4 ohm at 10 V -> 700 V, 1.4 ohm at 10 V, VGS +/-16 V
- R102: MPN (none) -> RT1206FRE07511KL; Manufacturer (none) -> Yageo
- R103: MPN (none) -> CR1206-FX-1053ELF; Manufacturer (none) -> Bourns
- R104: MPN (none) -> RCC120649R9FKEA; Manufacturer (none) -> Vishay
- R106, R143: MPN (none) -> CR1206-FX-1372ELF; Manufacturer (none) -> Bourns
- R107: MPN (none) -> CR1206-FX-1433ELF; Manufacturer (none) -> Bourns
- R108: MPN (none) -> RK73H2BLTD2002F; Manufacturer (none) -> KOA Speer
- R111: MPN (none) -> CRCW1206147KFKTA; Manufacturer (none) -> Vishay
- R117: MPN (none) -> RNCL1206FTR220; Manufacturer (none) -> SEI Stackpole
- R126, R131: MPN HHV-25FT-52-2M7 -> HHV-25FR-52-2M7
- R130: value 5.97k -> 3.0k; footprint Resistor_SMD:R_1206_3216Metric -> Resistor_SMD:R_0805_2012Metric; Function HV feedback, lower (453.3 V; 5.49k for 500 V: 492.8 V) -> HV feedback, lower 1 of 2 (2 x 3.0k: 451.0 V; 2 x 2.7k for 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; MPN (none) -> 292-3.0K-RC; Manufacturer (none) -> Xicon
- R135: Function HV monitor / OVP divider, middle (HV_SENSE 2.35 V at 453.3 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 -> HV monitor / OVP divider, middle (HV_SENSE 2.34 V at 451.0 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; MPN (none) -> ERJ-8ENF7871V; Manufacturer (none) -> Panasonic
- R140: value 6.19k -> 6.2k; Function HV monitor / OVP divider, lower (OVP trip 544.6 V) -> HV monitor / OVP divider, lower (OVP trip 543.7 V); MPN (none) -> CRCW12066K20FKEAC; Manufacturer (none) -> Vishay
- U101: value TPS54202 -> TPS54302; symbol Regulator_Switching:TPS54202DDC -> Regulator_Switching:TPS54302; MPN TPS54202DDCR -> TPS54302DDCR; Rating 4.5-28 V, 2 A -> 4.5-28 V, 3 A, 400 kHz
Connections:
- net GND: now also R144.2; no longer R130.2
- new net: R130.2, R144.1
Other:
- note added: "TPS54302, TI reference design (SLVSDG6C Fig. 7-1); 100k / 13.7k -> 4.95 V; UVLO 511k / 105k"
- note removed: "TPS54202, TI reference design (SLVSD26C Fig. 7-1); 100k / 13.7k -> 4.95 V; UVLO 511k / 105k"
