File: hardware/dekatron/mcu.kicad_sch (KiCad schematic)
At the start: 30 parts, among them J301 DISP, J302 NIX_LV, U301 RP2040-Zero

Commit message: Freeze the dekatron BOM to the Mouser order; substitutions; re-route
- ORDERED_PARTS in gen_schematics.py: exact manufacturer part numbers from
  Cart_Oct08_0432PM.xls (committed as the record), overriding design-time MPNs
- Backorder substitutions: TPS54302 (pin-compatible 5 V buck), IPD70R1K4P7S
  (700 V CoolMOS P7, replaces the EOL IPD50R1K4CE), MMSZ5262BT1G, BAT54S RFG
- C301 is the user's F91 tantalum: polarised symbol and EIA 3216-18 footprint
- E24 dividers: HV feedback 2 x 3.0k 0805 (451.0 V; 2 x 2.7k for 500 V),
  OVP lower 6.2k (543.7 V); simulations re-run, docs updated
- Router: exact own-pad clearance, D301 GND escape via kept out of the
  RP2040 no-via area (D301 anchored rotated), 0.3 mm GND repair links
- Full re-route, DRC clean (expected U106 mismatch, one starved thermal);
  fab outputs regenerated

Co-Authored-By: Claude Opus 5.5 <noreply@anthropic.com>
Parts:
- C301: footprint Capacitor_SMD:C_1206_3216Metric -> Capacitor_Tantalum_SMD:CP_EIA-3216-18_Kemet-A; symbol Device:C -> Device:C_Polarized; MPN (none) -> F911C106MAAAJ6; Manufacturer (none) -> KYOCERA AVX; Rating 16 V X7R -> 16 V tantalum, 1.5 ohm ESR
- C302, C303, C305: MPN (none) -> CC1206JPX7R9BB104; Manufacturer (none) -> Yageo
- C304: MPN (none) -> 12063C103JAT2A; Manufacturer (none) -> KYOCERA AVX
- D301, D302, D303, D304: MPN BAT54S -> BAT54S RFG; Manufacturer (none) -> Taiwan Semiconductor
- R302: MPN (none) -> ERJ-8ENF1202V; Manufacturer (none) -> Panasonic
Changed lines of the file:
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@@
 	(wire (pts (xy 121.92 60.96) (xy 124.46 60.96)) (stroke (width 0) (type default)))
 	(label "UART_TX" (at 124.46 60.96 0) (effects (font (size 1.27 1.27)) (justify left bottom)))
-	(symbol (lib_id "Device:C") (at 33.02 53.34 0) (unit 1) (body_style 1) (exclude_from_sim no) (in_bom yes) (on_board yes) (in_pos_files yes) (dnp no)
+	(symbol (lib_id "Device:C_Polarized") (at 33.02 53.34 0) (unit 1) (body_style 1) (exclude_from_sim no) (in_bom yes) (on_board yes) (in_pos_files yes) (dnp no)
 	  (property "Reference" "C301" (at 36.22 52.34 0) (show_name no) (do_not_autoplace no) (effects (font (size 1.27 1.27)) (justify left)))
 	  (property "Value" "10uF" (at 36.22 54.94 0) (show_name no) (do_not_autoplace no) (effects (font (size 1.27 1.27)) (justify left)))
-	  (property "Footprint" "Capacitor_SMD:C_1206_3216Metric" (at 33.02 53.34 0) (hide yes) (show_name no) (do_not_autoplace no) (effects (font (size 1.27 1.27)) (justify left)))
+	  (property "Footprint" "Capacitor_Tantalum_SMD:CP_EIA-3216-18_Kemet-A" (at 33.02 53.34 0) (hide yes) (show_name no) (do_not_autoplace no) (effects (font (size 1.27 1.27)) (justify left)))
 	  (property "Datasheet" "" (at 33.02 53.34 0) (hide yes) (show_name no) (do_not_autoplace no) (effects (font (size 1.27 1.27)) (justify left)))
-	  (property "Description" "Unpolarized capacitor" (at 33.02 53.34 0) (hide yes) (show_name no) (do_not_autoplace no) (effects (font (size 1.27 1.27)) (justify left)))
+	  (property "Description" "Polarized capacitor" (at 33.02 53.34 0) (hide yes) (show_name no) (do_not_autoplace no) (effects (font (size 1.27 1.27)) (justify left)))
 	  (property "Function" "5V_MCU bulk at the module" (at 33.02 53.34 0) (hide yes) (show_name no) (do_not_autoplace no) (effects (font (size 1.27 1.27)) (justify left)))
-	  (property "Rating" "16 V X7R" (at 33.02 53.34 0) (hide yes) (show_name no) (do_not_autoplace no) (effects (font (size 1.27 1.27)) (justify left)))
+	  (property "MPN" "F911C106MAAAJ6" (at 33.02 53.34 0) (hide yes) (show_name no) (do_not_autoplace no) (effects (font (size 1.27 1.27)) (justify left)))
+	  (property "Manufacturer" "KYOCERA AVX" (at 33.02 53.34 0) (hide yes) (show_name no) (do_not_autoplace no) (effects (font (size 1.27 1.27)) (justify left)))
+	  (property "Rating" "16 V tantalum, 1.5 ohm ESR" (at 33.02 53.34 0) (hide yes) (show_name no) (do_not_autoplace no) (effects (font (size 1.27 1.27)) (justify left)))
 	  (pin "1")
 	  (pin "2")
@@
 	  (property "Function" "3V3 bypass" (at 48.26 53.34 0) (hide yes) (show_name no) (do_not_autoplace no) (effects (font (size 1.27 1.27)) (justify left)))
 	  (property "Rating" "50 V X7R" (at 48.26 53.34 0) (hide yes) (show_name no) (do_not_autoplace no) (effects (font (size 1.27 1.27)) (justify left)))
+	  (property "Manufacturer" "Yageo" (at 48.26 53.34 0) (hide yes) (show_name no) (do_not_autoplace no) (effects (font (size 1.27 1.27)) (justify left)))
+	  (property "MPN" "CC1206JPX7R9BB104" (at 48.26 53.34 0) (hide yes) (show_name no) (do_not_autoplace no) (effects (font (size 1.27 1.27)) (justify left)))
 	  (pin "1")
 	  (pin "2")
@@
 	  (property "Description" "Vr 30V, If 200mA, Dual schottky barrier diode, in series, SOT-323" (at 55.88 160.02 0) (hide yes) (show_name no) (do_not_autoplace no) (effects (font (size 1.27 1.27)) (justify left)))
 	  (property "Function" "VIN_SENSE clamp to 3V3 / GND" (at 55.88 160.02 0) (hide yes) (show_name no) (do_not_autoplace no) (effects (font (size 1.27 1.27)) (justify left)))
-	  (property "MPN" "BAT54S" (at 55.88 160.02 0) (hide yes) (show_name no) (do_not_autoplace no) (effects (font (size 1.27 1.27)) (justify left)))
+	  (property "MPN" "BAT54S RFG" (at 55.88 160.02 0) (hide yes) (show_name no) (do_not_autoplace no) (effects (font (size 1.27 1.27)) (justify left)))
+	  (property "Manufacturer" "Taiwan Semiconductor" (at 55.88 160.02 0) (hide yes) (show_name no) (do_not_autoplace no) (effects (font (size 1.27 1.27)) (justify left)))
 	  (property "Rating" "30 V Schottky pair" (at 55.88 160.02 0) (hide yes) (show_name no) (do_not_autoplace no) (effects (font (size 1.27 1.27)) (justify left)))
 	  (pin "1")
@@
 	  (property "Function" "VIN_SENSE ADC sampling reservoir" (at 55.88 182.88 0) (hide yes) (show_name no) (do_not_autoplace no) (effects (font (size 1.27 1.27)) (justify left)))
 	  (property "Rating" "25 V X7R" (at 55.88 182.88 0) (hide yes) (show_name no) (do_not_autoplace no) (effects (font (size 1.27 1.27)) (justify left)))
+	  (property "Manufacturer" "Yageo" (at 55.88 182.88 0) (hide yes) (show_name no) (do_not_autoplace no) (effects (font (size 1.27 1.27)) (justify left)))
+	  (property "MPN" "CC1206JPX7R9BB104" (at 55.88 182.88 0) (hide yes) (show_name no) (do_not_autoplace no) (effects (font (size 1.27 1.27)) (justify left)))
 	  (pin "1")
 	  (pin "2")
@@
 	  (property "Function" "VIN_SENSE divider, lower (2.57 V at 24 V)" (at 45.72 182.88 0) (hide yes) (show_name no) (do_not_autoplace no) (effects (font (size 1.27 1.27)) (justify left)))
 	  (property "Rating" "1 %" (at 45.72 182.88 0) (hide yes) (show_name no) (do_not_autoplace no) (effects (font (size 1.27 1.27)) (justify left)))
+	  (property "Manufacturer" "Panasonic" (at 45.72 182.88 0) (hide yes) (show_name no) (do_not_autoplace no) (effects (font (size 1.27 1.27)) (justify left)))
+	  (property "MPN" "ERJ-8ENF1202V" (at 45.72 182.88 0) (hide yes) (show_name no) (do_not_autoplace no) (effects (font (size 1.27 1.27)) (justify left)))
 	  (pin "1")
 	  (pin "2")
@@
 	  (property "Description" "Vr 30V, If 200mA, Dual schottky barrier diode, in series, SOT-323" (at 106.68 160.02 0) (hide yes) (show_name no) (do_not_autoplace no) (effects (font (size 1.27 1.27)) (justify left)))
 	  (property "Function" "HV_SENSE clamp to 3V3 / GND" (at 106.68 160.02 0) (hide yes) (show_name no) (do_not_autoplace no) (effects (font (size 1.27 1.27)) (justify left)))
-	  (property "MPN" "BAT54S" (at 106.68 160.02 0) (hide yes) (show_name no) (do_not_autoplace no) (effects (font (size 1.27 1.27)) (justify left)))
+	  (property "MPN" "BAT54S RFG" (at 106.68 160.02 0) (hide yes) (show_name no) (do_not_autoplace no) (effects (font (size 1.27 1.27)) (justify left)))
+	  (property "Manufacturer" "Taiwan Semiconductor" (at 106.68 160.02 0) (hide yes) (show_name no) (do_not_autoplace no) (effects (font (size 1.27 1.27)) (justify left)))
 	  (property "Rating" "30 V Schottky pair" (at 106.68 160.02 0) (hide yes) (show_name no) (do_not_autoplace no) (effects (font (size 1.27 1.27)) (justify left)))
 	  (pin "1")
@@
 	  (property "Function" "HV_SENSE ADC sampling reservoir" (at 106.68 182.88 0) (hide yes) (show_name no) (do_not_autoplace no) (effects (font (size 1.27 1.27)) (justify left)))
 	  (property "Rating" "25 V X7R" (at 106.68 182.88 0) (hide yes) (show_name no) (do_not_autoplace no) (effects (font (size 1.27 1.27)) (justify left)))
+	  (property "Manufacturer" "KYOCERA AVX" (at 106.68 182.88 0) (hide yes) (show_name no) (do_not_autoplace no) (effects (font (size 1.27 1.27)) (justify left)))
+	  (property "MPN" "12063C103JAT2A" (at 106.68 182.88 0) (hide yes) (show_name no) (do_not_autoplace no) (effects (font (size 1.27 1.27)) (justify left)))
 	  (pin "1")
 	  (pin "2")
@@
 	  (property "Description" "Vr 30V, If 200mA, Dual schottky barrier diode, in series, SOT-323" (at 157.48 160.02 0) (hide yes) (show_name no) (do_not_autoplace no) (effects (font (size 1.27 1.27)) (justify left)))
 	  (property "Function" "RTN_SENSE clamp to 3V3 / GND" (at 157.48 160.02 0) (hide yes) (show_name no) (do_not_autoplace no) (effects (font (size 1.27 1.27)) (justify left)))
-	  (property "MPN" "BAT54S" (at 157.48 160.02 0) (hide yes) (show_name no) (do_not_autoplace no) (effects (font (size 1.27 1.27)) (justify left)))
+	  (property "MPN" "BAT54S RFG" (at 157.48 160.02 0) (hide yes) (show_name no) (do_not_autoplace no) (effects (font (size 1.27 1.27)) (justify left)))
+	  (property "Manufacturer" "Taiwan Semiconductor" (at 157.48 160.02 0) (hide yes) (show_name no) (do_not_autoplace no) (effects (font (size 1.27 1.27)) (justify left)))
 	  (property "Rating" "30 V Schottky pair" (at 157.48 160.02 0) (hide yes) (show_name no) (do_not_autoplace no) (effects (font (size 1.27 1.27)) (justify left)))
 	  (pin "1")
@@
 	  (property "Function" "RTN_SENSE ADC sampling reservoir" (at 157.48 182.88 0) (hide yes) (show_name no) (do_not_autoplace no) (effects (font (size 1.27 1.27)) (justify left)))
 	  (property "Rating" "25 V X7R" (at 157.48 182.88 0) (hide yes) (show_name no) (do_not_autoplace no) (effects (font (size 1.27 1.27)) (justify left)))
+	  (property "Manufacturer" "Yageo" (at 157.48 182.88 0) (hide yes) (show_name no) (do_not_autoplace no) (effects (font (size 1.27 1.27)) (justify left)))
+	  (property "MPN" "CC1206JPX7R9BB104" (at 157.48 182.88 0) (hide yes) (show_name no) (do_not_autoplace no) (effects (font (size 1.27 1.27)) (justify left)))
 	  (pin "1")
 	  (pin "2")
@@
 	  (property "Description" "Vr 30V, If 200mA, Dual schottky barrier diode, in series, SOT-323" (at 208.28 160.02 0) (hide yes) (show_name no) (do_not_autoplace no) (effects (font (size 1.27 1.27)) (justify left)))
 	  (property "Function" "NDX clamp to 3V3 / GND" (at 208.28 160.02 0) (hide yes) (show_name no) (do_not_autoplace no) (effects (font (size 1.27 1.27)) (justify left)))
-	  (property "MPN" "BAT54S" (at 208.28 160.02 0) (hide yes) (show_name no) (do_not_autoplace no) (effects (font (size 1.27 1.27)) (justify left)))
+	  (property "MPN" "BAT54S RFG" (at 208.28 160.02 0) (hide yes) (show_name no) (do_not_autoplace no) (effects (font (size 1.27 1.27)) (justify left)))
+	  (property "Manufacturer" "Taiwan Semiconductor" (at 208.28 160.02 0) (hide yes) (show_name no) (do_not_autoplace no) (effects (font (size 1.27 1.27)) (justify left)))
 	  (property "Rating" "30 V Schottky pair" (at 208.28 160.02 0) (hide yes) (show_name no) (do_not_autoplace no) (effects (font (size 1.27 1.27)) (justify left)))
 	  (pin "1")
